File: remoteid-esp32-s3/remoteid-esp32-s3.kicad_pcb (KiCad board)
At the start: 2 copper layers, 38.5 x 38.5 mm, 34 parts, among them J1 USB_C_Receptacle_USB2.0, J2 CAN, SW1 RESET, SW2 BOOT, U1 ESP32-S3-MINI-1, U2 SN65HVD230, U3 USBLC6-2SC6, U4 AMS1117-3.3

Commit message: updated
Parts:
- renumbered UART to J3
Routing:
- net GND: track 65.0 -> 49.1 mm, vias 33 -> 54
- net +3.3V: track 41.9 -> 52.4 mm, vias 2 -> 4
- added copper zone on F.Cu, net GND

Commit message: changes
Parts:
- removed C2: 0.1u, Capacitor_SMD:C_0603_1608Metric
- removed C8, C9: 22p, Capacitor_SMD:C_0603_1608Metric
- removed FB1: >1A, Capacitor_SMD:C_0603_1608Metric
- removed R6, R7: 22r, Resistor_SMD:R_0603_1608Metric
- removed U3: USBLC6-2SC6, Package_TO_SOT_SMD:SOT-23-6
- added D2: PRTR5V0U2X, Package_TO_SOT_SMD:SOT-143, F.Cu at (164.3, 80.4)
- C1: footprint Capacitor_SMD:C_0603_1608Metric -> Capacitor_SMD:C_0805_2012Metric
- C10: value 10u -> 10uF; footprint Capacitor_SMD:C_0603_1608Metric -> Capacitor_SMD:C_0805_2012Metric
- C11: value 4.7u -> 4.7uF; footprint Capacitor_SMD:C_0603_1608Metric -> Capacitor_SMD:C_0805_2012Metric
- C12: value 0.1uF -> 100nF; footprint Capacitor_SMD:C_0603_1608Metric -> Capacitor_SMD:C_0805_2012Metric
- C3, C5, C6, C7: value 0.1u -> 100nF; footprint Capacitor_SMD:C_0603_1608Metric -> Capacitor_SMD:C_0805_2012Metric
- C4: value 22u -> 22uF; footprint Capacitor_SMD:C_0603_1608Metric -> Capacitor_SMD:C_0805_2012Metric
- moved J3 16.3 mm to (153.8, 89.8), turned to 90 degrees
- moved C1 10.3 mm to (152.2, 61.2), turned to 90 degrees
- moved R1 7.02 mm to (176.3, 83.0), turned to 0 degrees
- moved C6 4.87 mm to (180.0, 66.4), turned to 0 degrees
- moved C7 4.83 mm to (179.2, 79.0), turned to 0 degrees
- moved FB2 4.63 mm to (161.7, 84.8), turned to 90 degrees
- moved RST 4.56 mm to (178.8, 70.6), turned to 180 degrees
- moved C3 4.20 mm to (163.5, 84.8), turned to 90 degrees
- moved C12 4.17 mm to (180.0, 64.2), turned to 180 degrees
- moved R2 3.97 mm to (167.9, 82.0)
- moved J1 3.53 mm to (170.1, 88.1)
- moved C11 2.53 mm to (152.2, 73.8), turned to 180 degrees
- moved C10 1.61 mm to (153.2, 85.6), turned to 0 degrees
- moved BOOT 1.56 mm to (178.8, 75.8), turned to 180 degrees
- moved U4 1.34 mm to (153.2, 79.8), turned to 0 degrees
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- renumbered SW2 to BOOT, SW1 to RST
Connections:
- C12 pad 1: /EN -> GND
- C12 pad 2: GND -> /EN
- J1 pad A6: /D+ -> /USB_D+
- J1 pad A7: /D- -> /USB_D-
- J1 pad B6: /D+ -> /USB_D+
- J1 pad B7: /D- -> /USB_D-
- J1 pad S1: Net-(C2-Pad2) -> GND
- U1 pad 23: Net-(R7-Pad2) -> /USB_D-
- U1 pad 24: Net-(R6-Pad2) -> /USB_D+
Routing:
- net /USB_D+: track 4.39 -> 27.0 mm, vias 0 -> 2
- net Net-(C2-Pad2): track 20.9 -> 0.00 mm
- net /USB_D-: track 4.35 -> 22.6 mm
- net /D-: track 4.88 -> 0.00 mm
- net /D+: track 4.47 -> 0.00 mm
- net VBUS: track 22.5 -> 18.3 mm, vias 2 -> 0
- net +5V: track 38.9 -> 42.9 mm
- net GND: track 49.1 -> 45.9 mm, vias 54 -> 55
- net /EN: track 15.4 -> 18.3 mm
- net Net-(J1-PadB5): track 3.03 -> 5.64 mm
- net Net-(R6-Pad2): track 2.43 -> 0.00 mm
- net Net-(R7-Pad2): track 2.28 -> 0.00 mm
- net /UART_TX: track 19.4 -> 21.1 mm
- net +3.3V: track 52.4 -> 50.7 mm, vias 4 -> 2
- net /UART_RX: track 21.5 -> 20.0 mm
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- added copper zone on F.Cu, net +3.3V

Commit message: changes
Parts:
- removed BOOT: BOOT, Autrik:Alps_SKRK
- removed RST: RESET, Autrik:Alps_SKRK
- J2, J3: footprint Connector_PinSocket_2.54mm:PinSocket_1x04_P2.54mm_Vertical -> Connector_JST:JST_GH_SM04B-GHS-TB_1x04-1MP_P1.25mm_Horizontal
- moved J2 3.84 mm to (146.4, 67.0), turned to -90 degrees
- moved J3 3.80 mm to (157.6, 89.9), turned to 0 degrees
Routing:
- net +5V: track 42.9 -> 44.6 mm, vias 0 -> 1
- net GND: track 45.9 -> 44.1 mm, vias 55 -> 54
Other:
- board text added: "RemoteID-v1.2 Designed by Autrik UG"
