File: remoteid-esp32-s3/remoteid-esp32-s3.kicad_sch (KiCad schematic)
At the start: 34 parts, among them J1 USB_C_Receptacle_USB2.0, J2 CAN, J3 UART, SW1 RESET, SW2 BOOT, U1 ESP32-S3-MINI-1, U2 SN65HVD230, U3 USBLC6-2SC6, U4 AMS1117-3.3

Commit message: updated
Parts:
- C10: value 10u -> 10uF
- C11: value 4.7u -> 4.7uF
- C12: value 0.1uF -> 100nF
- C2, C3, C5, C6, C7: value 0.1u -> 100nF; LCSC (none) -> C14663; MPN (none) -> C14663
- C4: value 22u -> 22uF
- C8, C9: value 22p -> 22pF
- D1: LCSC (none) -> C205445; MPN (none) -> C205445
- FB1, FB2: LCSC (none) -> C85831; MPN (none) -> C85831
- J1: LCSC (none) -> C165948; MPN (none) -> C165948
- SW1, SW2: LCSC (none) -> C115357; MPN (none) -> C115357
- U1: LCSC (none) -> C2980299; MPN (none) -> C2980299
- U2: LCSC (none) -> C12084; MPN (none) -> C12084
- U3: LCSC (none) -> C558442; MPN (none) -> C558442
- U4: LCSC (none) -> C6186; MPN (none) -> C6186
Other:
- title: (none) -> Remote ID ESP32 S3

Commit message: changes
Parts:
- removed C2: 100nF, Capacitor_SMD:C_0603_1608Metric, symbol Device:C
- removed C8, C9: 22pF, Capacitor_SMD:C_0603_1608Metric, symbol Device:C
- removed FB1: >1A, C_0603_1608Metric, symbol Device:FerriteBead_Small
- removed R6, R7: 22r, Resistor_SMD:R_0603_1608Metric, symbol Device:R
- removed U3: USBLC6-2SC6, Package_TO_SOT_SMD:SOT-23-6, symbol Power_Protection:USBLC6-2SC6
- added D2: PRTR5V0U2X, Package_TO_SOT_SMD:SOT-143, symbol Power_Protection:PRTR5V0U2X
- C1, C10, C11, C12, C3, C4, C5, C6, C7: footprint Capacitor_SMD:C_0603_1608Metric -> Capacitor_SMD:C_0805_2012Metric
Connections:
- net D+ is gone; now on net USB_D+: J1.A6 (D+), J1.B6 (D+)
- net D- is gone; now on net USB_D-: J1.A7 (D-), J1.B7 (D-)
- net EN: now also C12.2; no longer C12.1
- net GND: now also C12.1, J1.S1 (SHIELD), D2.1 (GND); no longer C12.2
- net USB_D+: now also U1.24 (GPIO20/U1CTS/ADC2_CH9/CLK_OUT1/USB_D+), D2.2 (I/O1)
- net USB_D-: now also U1.23 (GPIO19/U1RTS/ADC2_CH8/CLK_OUT2/USB_D-), D2.3 (I/O2)
- net VBUS: now also D2.4 (VCC)
Other:
- moved on the sheet: C1, C10, C11, C12, C3, C4, C5, C6, C7, D1, FB2, H1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

Commit message: changes
Parts:
- J2, J3: footprint Connector_PinSocket_2.54mm:PinSocket_1x04_P2.54mm_Vertical -> Connector_JST:JST_GH_SM04B-GHS-TB_1x04-1MP_P1.25mm_Horizontal
Changed lines of the file:
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@@
       (effects (font (size 1.27 1.27)) (justify left))
     )
-    (property "Footprint" "Connector_PinSocket_2.54mm:PinSocket_1x04_P2.54mm_Vertical" (id 2) (at 370.84 124.46 0)
+    (property "Footprint" "Connector_JST:JST_GH_SM04B-GHS-TB_1x04-1MP_P1.25mm_Horizontal" (id 2) (at 370.84 124.46 0)
       (effects (font (size 1.27 1.27)) hide)
     )
@@
       (effects (font (size 1.27 1.27)) (justify left))
     )
-    (property "Footprint" "Connector_PinSocket_2.54mm:PinSocket_1x04_P2.54mm_Vertical" (id 2) (at 372.11 95.25 0)
+    (property "Footprint" "Connector_JST:JST_GH_SM04B-GHS-TB_1x04-1MP_P1.25mm_Horizontal" (id 2) (at 372.11 95.25 0)
       (effects (font (size 1.27 1.27)) hide)
     )
@@
     )
     (path "/b5c93212-d51a-4e09-888e-c06703f74140"
-      (reference "J2") (unit 1) (value "CAN") (footprint "Connector_PinSocket_2.54mm:PinSocket_1x04_P2.54mm_Vertical")
+      (reference "J2") (unit 1) (value "CAN") (footprint "Connector_JST:JST_GH_SM04B-GHS-TB_1x04-1MP_P1.25mm_Horizontal")
     )
     (path "/f4ea0a4d-4f31-4d0b-b8e1-eff7ab74755d"
-      (reference "J3") (unit 1) (value "UART") (footprint "Connector_PinSocket_2.54mm:PinSocket_1x04_P2.54mm_Vertical")
+      (reference "J3") (unit 1) (value "UART") (footprint "Connector_JST:JST_GH_SM04B-GHS-TB_1x04-1MP_P1.25mm_Horizontal")
     )
     (path "/51e51ca2-a6d6-4d67-b20d-8a733565053b"
